Commit message: changee

File: description/robot.urdf.xacro (robot description, xacro)
@@ -1,4 +1,4 @@
 <?xml version="1.0"?>
-<robot xmlns:xacro="http://www.ros.org/wiki/xacro"  name="robot">
+<robot xmlns:xacro="http://www.ros.org/wiki/xacro" name="robot">
      <xacro:include filename="robot_core.xacro" />
      <xacro:include filename="colors.xacro" />

File: description/robot_core.xacro (robot description, xacro)
@@ -2,18 +2,84 @@
 <robot xmlns:xacro="http://www.ros.org/wiki/xacro">
     <link name="base_link">
-        <joint name="chassis_joint" type="fixed">
-            <parent link="base_link" />
-            <child link="chassic" />
-            <origin xyz="-0.1 0 0" />
-        </joint>
-        <link name="chassis">
-            <visual>
-                <origin xyz="0.9 0 0.6" rpy="0 0 0 " />
-                <geometry>
-                    <box size="0.18 0.16 0.12" />
-                </geometry>
-                <material name="white" />
-            </visual>
-        </link>
     </link>
-</robot>å
+    <joint name="chassis_joint" type="fixed">
+        <parent link="base_link" />
+        <child link="chassis" />
+        <origin xyz="-0.09 0 0" />
+    </joint>
+    <link name="chassis">
+        <visual>
+            <origin xyz="0 0 0.03" rpy="0 0 0 " />
+            <geometry>
+                <box size="0.18 0.16 0.12" />
+            </geometry>
+            <material name="white" />
+        </visual>
+        <collision>
+            <origin xyz="0 0 0.03" rpy="0 0 0 " />
+            <geometry>
+                <box size="0.18 0.16 0.12" />
+            </geometry>
+        </collision>
+    </link>
+    <!-- left wheel-->
+    <joint name="left_wheel_joint" type="continuous">
+        <parent link="base_link" />
+        <child link="left_wheel" />
+        <origin xyz="-0.08 0.08 0" rpy="-${pi/2} 0 0" />
+        <axis xyz="0 0 1" />
+    </joint>
+    <link name="left_wheel">
+        <visual>
+            <geometry>
+                <cylinder length="0.025" radius="0.0325" />
+            </geometry>
+            <material name="blue" />
+        </visual>
+    </link>
+    <!-- right wheel-->
+    <joint name="right_wheel_joint" type="continuous">
+        <parent link="base_link" />
+        <child link="right_wheel" />
+        <origin xyz="-0.08 -0.08 0" rpy="-${pi/2} 0 0" />
+        <axis xyz="0 0 -1" />
+    </joint>
+    <link name="right_wheel">
+        <visual>
+            <geometry>
+                <cylinder length="0.025" radius="0.0325" />
+            </geometry>
+            <material name="blue" />
+        </visual>
+    </link>
+    <!--front
+    caster wheel-->
+    <joint name="front_caster_wheel_joint" type="fixed">
+        <parent link="chassis" />
+        <child link="front_caster_wheel" />
+        <origin xyz="-0.08 0 -0.0325" rpy="0 0 0" />
+    </joint>
+    <link name="front_caster_wheel">
+        <visual>
+            <geometry>
+                <sphere radius="0.0065" />
+            </geometry>
+            <material name="black" />
+        </visual>
+    </link>
+    <!--back
+    caster wheel-->
+    <joint name="back_caster_wheel_joint" type="fixed">
+        <parent link="chassis" />
+        <child link="back_caster_wheel" />
+        <origin xyz="0.08 0 -0.0325" rpy="0 0 0" />
+    </joint>
+    <link name="back_caster_wheel">
+        <visual>
+            <geometry>
+                <sphere radius="0.0065" />
+            </geometry>
+            <material name="black" />
+        </visual>
+    </link>
+</robot>

Commit message: added collision, inertial and gazebo control

File: description/robot.urdf.xacro (robot description, xacro)
@@ -1,4 +1,5 @@
 <?xml version="1.0"?>
 <robot xmlns:xacro="http://www.ros.org/wiki/xacro" name="robot">
+     <xacro:include filename='inertial_macros.xacro' />
      <xacro:include filename="robot_core.xacro" />
      <xacro:include filename="colors.xacro" />

File: description/robot_core.xacro (robot description, xacro)
@@ -22,5 +22,11 @@
             </geometry>
         </collision>
+        <xacro:inertial_box mass="0.92" x="0" y="0" z="0.03">
+            <origin xyz="0.15 0 0.075" rpy="0 0 0" />
+        </xacro:inertial_box>
     </link>
+    <gazebo reference="chassis">
+        <material>Gazebo/White</material>
+    </gazebo>
     <!-- left wheel-->
     <joint name="left_wheel_joint" type="continuous">
@@ -37,5 +43,11 @@
             <material name="blue" />
         </visual>
+        <xacro:inertial_cylinder mass="0.05" length="0.025" radius="0.0325">
+            <origin xyz="0 0 0" rpy="0 0 0" />
+        </xacro:inertial_cylinder>
     </link>
+    <gazebo reference="left_wheel">
+        <material>Gazebo/Blue</material>
+    </gazebo>
     <!-- right wheel-->
     <joint name="right_wheel_joint" type="continuous">
@@ -52,5 +64,11 @@
             <material name="blue" />
         </visual>
+        <xacro:inertial_cylinder mass="0.05" length="0.025" radius="0.0325">
+            <origin xyz="0 0 0" rpy="0 0 0" />
+        </xacro:inertial_cylinder>
     </link>
+    <gazebo reference="right_wheel">
+        <material>Gazebo/Blue</material>
+    </gazebo>
     <!--front
     caster wheel-->
@@ -67,5 +85,13 @@
             <material name="black" />
         </visual>
+        <xacro:inertial_sphere mass="0.01" radius="0.008">
+            <origin xyz="-0.08 0 -0.0325" rpy="0 0 0" />
+        </xacro:inertial_sphere>
     </link>
+    <gazebo reference="front_caster_wheel">
+        <material>Gazebo/Black</material>
+        <mu1 value="0.001" />
+        <mu2 value="0.001" />
+    </gazebo>
     <!--back
     caster wheel-->
@@ -82,4 +108,12 @@
             <material name="black" />
         </visual>
+        <xacro:inertial_sphere mass="0.01" radius="0.008">
+            <origin xyz="-0.08 0 -0.0325" rpy="0 0 0" />
+        </xacro:inertial_sphere>
     </link>
+    <gazebo reference="back_caster_wheel">
+        <material>Gazebo/Black</material>
+        <mu1 value="0.001" />
+        <mu2 value="0.001" />
+    </gazebo>
 </robot>
