Commit message: change

File: description/robot_core.xacro (robot description, xacro)
@@ -1,5 +1,19 @@
 <?xml version="1.0"?>
 <robot xmlns:xacro="http://www.ros.org/wiki/xacro">
-<link name="base_link">
-</link>
-</robot>
+    <link name="base_link">
+        <joint name="chassis_joint" type="fixed">
+            <parent link="base_link" />
+            <child link="chassic" />
+            <origin xyz="-0.1 0 0" />
+        </joint>
+        <link name="chassis">
+            <visual>
+                <origin xyz="0.9 0 0.6" rpy="0 0 0 " />
+                <geometry>
+                    <box size="0.18 0.16 0.12" />
+                </geometry>
+                <material name="white" />
+            </visual>
+        </link>
+    </link>
+</robot>å

Commit message: fixed chassis inertial

File: description/robot_core.xacro (robot description, xacro)
@@ -23,5 +23,5 @@
         </collision>
         <xacro:inertial_box mass="0.92" x="0" y="0" z="0.03">
-            <origin xyz="0.15 0 0.075" rpy="0 0 0" />
+            <origin xyz="0 0 0.03" rpy="0 0 0 " />
         </xacro:inertial_box>
     </link>
@@ -109,5 +109,5 @@
         </visual>
         <xacro:inertial_sphere mass="0.01" radius="0.008">
-            <origin xyz="-0.08 0 -0.0325" rpy="0 0 0" />
+            <origin xyz="0.08 0 -0.0325" rpy="0 0 0" />
         </xacro:inertial_sphere>
     </link>

Commit message: Finished the URDF for chassis finally

File: description/robot_core.xacro (robot description, xacro)
@@ -10,5 +10,5 @@
     <link name="chassis">
         <visual>
-            <origin xyz="0 0 0.03" rpy="0 0 0 " />
+            <origin xyz="0 0 0.04" rpy="0 0 0 " />
             <geometry>
                 <box size="0.18 0.16 0.12" />
@@ -17,11 +17,11 @@
         </visual>
         <collision>
-            <origin xyz="0 0 0.03" rpy="0 0 0 " />
+            <origin xyz="0 0 0.04" rpy="0 0 0 " />
             <geometry>
                 <box size="0.18 0.16 0.12" />
             </geometry>
         </collision>
-        <xacro:inertial_box mass="0.92" x="0" y="0" z="0.03">
-            <origin xyz="0 0 0.03" rpy="0 0 0 " />
+        <xacro:inertial_box mass="0.92" x="0.18" y="0.16" z="0.12">
+            <origin xyz="0 0 0.04" rpy="0 0 0 " />
         </xacro:inertial_box>
     </link>
@@ -33,5 +33,5 @@
         <parent link="base_link" />
         <child link="left_wheel" />
-        <origin xyz="-0.08 0.08 0" rpy="-${pi/2} 0 0" />
+        <origin xyz="-0.09 0.09225 0" rpy="-${pi/2} 0 0" />
         <axis xyz="0 0 1" />
     </joint>
@@ -46,4 +46,9 @@
             <origin xyz="0 0 0" rpy="0 0 0" />
         </xacro:inertial_cylinder>
+        <collision>
+            <geometry>
+                <cylinder length="0.025" radius="0.0325" />
+            </geometry>
+        </collision>
     </link>
     <gazebo reference="left_wheel">
@@ -54,5 +59,5 @@
         <parent link="base_link" />
         <child link="right_wheel" />
-        <origin xyz="-0.08 -0.08 0" rpy="-${pi/2} 0 0" />
+        <origin xyz="-0.09 -0.09225 0" rpy="-${pi/2} 0 0" />
         <axis xyz="0 0 -1" />
     </joint>
@@ -64,4 +69,9 @@
             <material name="blue" />
         </visual>
+        <collision>
+            <geometry>
+                <cylinder length="0.025" radius="0.0325" />
+            </geometry>
+        </collision>
         <xacro:inertial_cylinder mass="0.05" length="0.025" radius="0.0325">
             <origin xyz="0 0 0" rpy="0 0 0" />
@@ -76,15 +86,20 @@
         <parent link="chassis" />
         <child link="front_caster_wheel" />
-        <origin xyz="-0.08 0 -0.0325" rpy="0 0 0" />
+        <origin xyz="-0.08 0 -0.0225" rpy="0 0 0" />
     </joint>
     <link name="front_caster_wheel">
         <visual>
             <geometry>
-                <sphere radius="0.0065" />
+                <sphere radius="0.008" />
             </geometry>
             <material name="black" />
         </visual>
+        <collision>
+            <geometry>
+                <sphere radius="0.008" />
+            </geometry>
+        </collision>
         <xacro:inertial_sphere mass="0.01" radius="0.008">
-            <origin xyz="-0.08 0 -0.0325" rpy="0 0 0" />
+            <origin xyz="-0.08 0 -0.0225" rpy="0 0 0" />
         </xacro:inertial_sphere>
     </link>
@@ -99,15 +114,20 @@
         <parent link="chassis" />
         <child link="back_caster_wheel" />
-        <origin xyz="0.08 0 -0.0325" rpy="0 0 0" />
+        <origin xyz="0.08 0 -0.0225" rpy="0 0 0" />
     </joint>
     <link name="back_caster_wheel">
         <visual>
             <geometry>
-                <sphere radius="0.0065" />
+                <sphere radius="0.008" />
             </geometry>
             <material name="black" />
         </visual>
+        <collision>
+            <geometry>
+                <sphere radius="0.008" />
+            </geometry>
+        </collision>
         <xacro:inertial_sphere mass="0.001" radius="0.008">
-            <origin xyz="0.08 0 -0.0325" rpy="0 0 0" />
+            <origin xyz="0.08 0 -0.0225" rpy="0 0 0" />
         </xacro:inertial_sphere>
     </link>

Commit message: Finished integrating ros control with gazebo, fixed gazebo clock rateand wheel drift issue

File: description/robot_core.xacro (robot description, xacro)
@@ -48,5 +48,5 @@
         <collision>
             <geometry>
-                <cylinder length="0.025" radius="0.0325" />
+                <sphere radius="0.0325" />
             </geometry>
         </collision>
@@ -71,5 +71,5 @@
         <collision>
             <geometry>
-                <cylinder length="0.025" radius="0.0325" />
+                <sphere radius="0.0325" />
             </geometry>
         </collision>
